File: pcb/hackpad.kicad_pcb (KiCad board)
At the start: 2 copper layers, 85 x 80 mm, 32 parts, among them J1 OLED Connection, SW1 SW_Push, SW11 RotaryEncoder_Switch, SW2 SW_Push, SW3 SW_Push, SW4 SW_Push, SW5 SW_Push, SW6 SW_Push, SW7 SW_Push, SW8 SW_Push

Commit message: edit pcb
Parts:
- removed anime: LOGO, Images:anime

Commit message: add drill files to gerbers.zip
Other:
- board text added: "JLCJLCJLCJLC"
Changed lines of the file:
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@@
 		(layer "Edge.Cuts")
+	)
+	(gr_text "JLCJLCJLCJLC"
+		(at 144.7 146.2 0)
+		(layer "B.SilkS")
+		(effects
+			(font
+				(size 1 1)
+				(thickness 0.1)
+			)
+			(justify left bottom mirror)
+		)
 	)
 	(segment
